File: LED Watch - empty RGB version.kicad_sch (KiCad schematic)
At the start: 139 parts, among them J1 AVR-ISP-6, J2 Lipo, J3 Coin Cell, SW1 SW_DPST, SW2 SW_DPST, U1 ATmega165PA-A, U10 B39D3RGB-F6C0001HOU1930, U100 B39D3RGB-F6C0001HOU1930, U101 B39D3RGB-F6C0001HOU1930, U102 B39D3RGB-F6C0001HOU1930, U103 B39D3RGB-F6C0001HOU1930, U104 B39D3RGB-F6C0001HOU1930, U105 B39D3RGB-F6C0001HOU1930, U106 B39D3RGB-F6C0001HOU1930, U107 B39D3RGB-F6C0001HOU1930, U108 B39D3RGB-F6C0001HOU1930, U109 B39D3RGB-F6C0001HOU1930, U11 B39D3RGB-F6C0001HOU1930, U110 B39D3RGB-F6C0001HOU1930, U111 B39D3RGB-F6C0001HOU1930, U112 B39D3RGB-F6C0001HOU1930, U113 B39D3RGB-F6C0001HOU1930, U114 B39D3RGB-F6C0001HOU1930, U115 B39D3RGB-F6C0001HOU1930, U116 B39D3RGB-F6C0001HOU1930, U117 B39D3RGB-F6C0001HOU1930, U118 B39D3RGB-F6C0001HOU1930, U119 B39D3RGB-F6C0001HOU1930, U12 B39D3RGB-F6C0001HOU1930, U120 B39D3RGB-F6C0001HOU1930, U121 B39D3RGB-F6C0001HOU1930, U122 B39D3RGB-F6C0001HOU1930, U123 B39D3RGB-F6C0001HOU1930, U124 B39D3RGB-F6C0001HOU1930, U125 B39D3RGB-F6C0001HOU1930, U126 B39D3RGB-F6C0001HOU1930, U127 B39D3RGB-F6C0001HOU1930, U128 B39D3RGB-F6C0001HOU1930, U129 B39D3RGB-F6C0001HOU1930, U13 B39D3RGB-F6C0001HOU1930, U130 B39D3RGB-F6C0001HOU1930, U131 B39D3RGB-F6C0001HOU1930, U132 B39D3RGB-F6C0001HOU1930, U133 B39D3RGB-F6C0001HOU1930, U134 BMI160, U14 B39D3RGB-F6C0001HOU1930, U15 B39D3RGB-F6C0001HOU1930, U16 B39D3RGB-F6C0001HOU1930, U17 B39D3RGB-F6C0001HOU1930, U18 B39D3RGB-F6C0001HOU1930, U19 B39D3RGB-F6C0001HOU1930, U2 B39D3RGB-F6C0001HOU1930, U20 B39D3RGB-F6C0001HOU1930, U21 B39D3RGB-F6C0001HOU1930, U22 B39D3RGB-F6C0001HOU1930, U23 B39D3RGB-F6C0001HOU1930, U24 B39D3RGB-F6C0001HOU1930, U25 B39D3RGB-F6C0001HOU1930, U26 B39D3RGB-F6C0001HOU1930, U27 B39D3RGB-F6C0001HOU1930, U28 B39D3RGB-F6C0001HOU1930, U29 B39D3RGB-F6C0001HOU1930, U3 B39D3RGB-F6C0001HOU1930, U30 B39D3RGB-F6C0001HOU1930, U31 B39D3RGB-F6C0001HOU1930, U32 B39D3RGB-F6C0001HOU1930, U33 B39D3RGB-F6C0001HOU1930, U34 B39D3RGB-F6C0001HOU1930, U35 B39D3RGB-F6C0001HOU1930, U36 B39D3RGB-F6C0001HOU1930, U37 B39D3RGB-F6C0001HOU1930, U38 B39D3RGB-F6C0001HOU1930, U39 B39D3RGB-F6C0001HOU1930, U4 B39D3RGB-F6C0001HOU1930, U40 B39D3RGB-F6C0001HOU1930, U41 B39D3RGB-F6C0001HOU1930, U42 B39D3RGB-F6C0001HOU1930, U43 B39D3RGB-F6C0001HOU1930, U44 B39D3RGB-F6C0001HOU1930, U45 B39D3RGB-F6C0001HOU1930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

Commit message: adjusted clocking and spacings.. ready for routing
Parts:
- J1: footprint (none) -> Connector_JST:JST_SH_BM05B-SRSS-TB_1x05-1MP_P1.00mm_Vertical
Changed lines of the file:
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@@
 			)
 		)
-		(property "Footprint" ""
+		(property "Footprint" "Connector_JST:JST_SH_BM05B-SRSS-TB_1x05-1MP_P1.00mm_Vertical"
 			(at 46.99 232.41 90)
 			(effects

Commit message: adjusted clocking and spacings.. ready for routing again
Parts:
- removed U1: ATmega165PA-A, Package_QFP:TQFP-64_14x14mm_P0.8mm, symbol MCU_Microchip_ATmega:ATmega165PA-A
- added U135: ATmega165PA-M, Package_DFN_QFN:QFN-64-1EP_9x9mm_P0.5mm_EP5.4x5.4mm, symbol MCU_Microchip_ATmega:ATmega165PA-M
- added Y1: Crystal, Crystal:Crystal_SMD_3215-2Pin_3.2x1.5mm, symbol Device:Crystal
Connections:
- net B1: now also U135.49 (PA2)
- net B2: now also U135.46 (PA5)
- net B3: now also U135.10 (PB0)
- net B4: now also U135.13 (PB3)
- net B5: now also U135.16 (PB6)
- net B6: now also U135.36 (PC1)
- net G1: now also U135.50 (PA1)
- net G2: now also U135.47 (PA4)
- net G3: now also U135.44 (PA7)
- net G4: now also U135.12 (PB2)
- net G5: now also U135.15 (PB5)
- net G6: now also U135.35 (PC0)
- net Hour1: now also U3.1, U4.1, U5.1, U6.1, U7.1, U135.37 (PC2)
- net Hour2: now also U10.1, U11.1, U12.1, U13.1, U9.1, U135.38 (PC3)
- net Minute1: now also U15.1, U16.1, U17.1, U18.1, U19.1, U135.39 (PC4)
- net Minute10: now also U69.1, U70.1, U71.1, U72.1, U73.1, U135.56 (PF5)
- net Minute2: now also U21.1, U22.1, U23.1, U24.1, U25.1, U135.40 (PC5)
- net Minute3: now also U27.1, U28.1, U29.1, U30.1, U31.1, U135.41 (PC6)
- net Minute4: now also U33.1, U34.1, U35.1, U36.1, U37.1, U135.42 (PC7)
- net Minute5: now also U39.1, U40.1, U41.1, U42.1, U43.1, U135.27 (PD2)
- net Minute6: now also U45.1, U46.1, U47.1, U48.1, U49.1, U135.28 (PD3)
- net Minute7: now also U51.1, U52.1, U53.1, U54.1, U55.1, U135.29 (PD4)
- net Minute8: now also U57.1, U58.1, U59.1, U60.1, U61.1, U135.30 (PD5)
- net Minute9: now also U63.1, U64.1, U65.1, U66.1, U67.1, U135.57 (PF4)
- net R1: now also U135.51 (PA0)
- net R2: now also U135.48 (PA3)
- net R3: now also U135.45 (PA6)
- net R4: now also U135.11 (PB1)
- net R5: now also U135.14 (PB4)
- net R6: now also U135.17 (PB7)
- net Second1: now also U75.1, U76.1, U77.1, U78.1, U79.1, U135.4 (PE2)
- net Second10: now also U135.18 (PG3)
- net Second2: now also U81.1, U82.1, U83.1, U84.1, U85.1, U135.5 (PE3)
- net Second3: now also U87.1, U88.1, U89.1, U90.1, U91.1, U135.6 (PE4)
- net Second4: now also U93.1, U94.1, U95.1, U96.1, U97.1, U135.7 (PE5)
- net Second5: now also U100.1, U101.1, U102.1, U103.1, U99.1, U135.8 (PE6)
- net Second6: now also U105.1, U106.1, U107.1, U108.1, U109.1, U135.9 (PE7)
- net Second7: now also U111.1, U112.1, U113.1, U114.1, U115.1, U135.33 (PG0)
- net Second8: now also U117.1, U118.1, U119.1, U120.1, U121.1, U135.34 (PG1)
- net Second9: now also U123.1, U124.1, U125.1, U126.1, U127.1, U135.43 (PG2)
- net at J1.2 (VCC), J2.1 (Pin_1), J3.1 (Pin_1)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: now also U135.21 (VCC), U135.52 (VCC)
- net at J1.5 (~{RST}): now also U135.20 (PG5/~{RESET})
- net at J1.6 (GND), J2.2 (Pin_2), J3.2 (Pin_2)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: now also U135.22 (GND), U135.53 (GND), U135.63 (GND), U135.65 (GND)
- net at SW2.1: now also U135.59 (PF2)
- net at SW2.2: now also U135.58 (PF3)
- net at U134.13 (SCx): now also U135.2 (PE0)
- net at U134.4 (INT1): now also U135.26 (PD1)
- net at U134.14 (SDx): now also U135.3 (PE1)
- net at SW1.2: now also U135.60 (PF1)
- net at SW1.1: now also U135.61 (PF0)
- new net: U135.31 (PD6), Y1.1
- new net: U135.32 (PD7), Y1.2
