File: _autosave-LED Watch.kicad_sch (KiCad schematic)
At the start: 142 parts, among them J1 AVR-ISP-6, J2 Lipo, J3 Coin Cell, SW1 SW_DPST, SW2 SW_DPST, U10 B39D3RGB-F6C0001HOU1930, U100 B39D3RGB-F6C0001HOU1930, U101 B39D3RGB-F6C0001HOU1930, U102 B39D3RGB-F6C0001HOU1930, U103 B39D3RGB-F6C0001HOU1930, U104 B39D3RGB-F6C0001HOU1930, U105 B39D3RGB-F6C0001HOU1930, U106 B39D3RGB-F6C0001HOU1930, U107 B39D3RGB-F6C0001HOU1930, U108 B39D3RGB-F6C0001HOU1930, U109 B39D3RGB-F6C0001HOU1930, U11 B39D3RGB-F6C0001HOU1930, U110 B39D3RGB-F6C0001HOU1930, U111 B39D3RGB-F6C0001HOU1930, U112 B39D3RGB-F6C0001HOU1930, U113 B39D3RGB-F6C0001HOU1930, U114 B39D3RGB-F6C0001HOU1930, U115 B39D3RGB-F6C0001HOU1930, U116 B39D3RGB-F6C0001HOU1930, U117 B39D3RGB-F6C0001HOU1930, U118 B39D3RGB-F6C0001HOU1930, U119 B39D3RGB-F6C0001HOU1930, U12 B39D3RGB-F6C0001HOU1930, U120 B39D3RGB-F6C0001HOU1930, U121 B39D3RGB-F6C0001HOU1930, U122 B39D3RGB-F6C0001HOU1930, U123 B39D3RGB-F6C0001HOU1930, U124 B39D3RGB-F6C0001HOU1930, U125 B39D3RGB-F6C0001HOU1930, U126 B39D3RGB-F6C0001HOU1930, U127 B39D3RGB-F6C0001HOU1930, U128 B39D3RGB-F6C0001HOU1930, U129 B39D3RGB-F6C0001HOU1930, U13 B39D3RGB-F6C0001HOU1930, U130 B39D3RGB-F6C0001HOU1930, U131 B39D3RGB-F6C0001HOU1930, U132 B39D3RGB-F6C0001HOU1930, U133 B39D3RGB-F6C0001HOU1930, U134 BMI160, U135 ATmega165PA-M, U14 B39D3RGB-F6C0001HOU1930, U15 B39D3RGB-F6C0001HOU1930, U16 B39D3RGB-F6C0001HOU1930, U17 B39D3RGB-F6C0001HOU1930, U18 B39D3RGB-F6C0001HOU1930, U19 B39D3RGB-F6C0001HOU1930, U2 B39D3RGB-F6C0001HOU1930, U20 B39D3RGB-F6C0001HOU1930, U21 B39D3RGB-F6C0001HOU1930, U22 B39D3RGB-F6C0001HOU1930, U23 B39D3RGB-F6C0001HOU1930, U24 B39D3RGB-F6C0001HOU1930, U25 B39D3RGB-F6C0001HOU1930, U26 B39D3RGB-F6C0001HOU1930, U27 B39D3RGB-F6C0001HOU1930, U28 B39D3RGB-F6C0001HOU1930, U29 B39D3RGB-F6C0001HOU1930, U3 B39D3RGB-F6C0001HOU1930, U30 B39D3RGB-F6C0001HOU1930, U31 B39D3RGB-F6C0001HOU1930, U32 B39D3RGB-F6C0001HOU1930, U33 B39D3RGB-F6C0001HOU1930, U34 B39D3RGB-F6C0001HOU1930, U35 B39D3RGB-F6C0001HOU1930, U36 B39D3RGB-F6C0001HOU1930, U37 B39D3RGB-F6C0001HOU1930, U38 B39D3RGB-F6C0001HOU1930, U39 B39D3RGB-F6C0001HOU1930, U4 B39D3RGB-F6C0001HOU1930, U40 B39D3RGB-F6C0001HOU1930, U41 B39D3RGB-F6C0001HOU1930, U42 B39D3RGB-F6C0001HOU1930, U43 B39D3RGB-F6C0001HOU1930, U44 B39D3RGB-F6C0001HOU1930, U45 B39D3RGB-F6C0001HOU1930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

Commit message: added caps.. still unsuccessful routing
Other:
- moved on the sheet: C1, C2
Changed lines of the file:
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@@
 	)
 	(junction
-		(at 119.38 196.85)
-		(diameter 0)
-		(color 0 0 0 0)
-	)
-	(junction
 		(at 342.9 106.68)
 		(diameter 0)
@@
 	)
 	(junction
+		(at 107.95 196.85)
+		(diameter 0)
+		(color 0 0 0 0)
+	)
+	(junction
 		(at 209.55 152.4)
 		(diameter 0)
@@
 	)
 	(junction
-		(at 64.77 204.47)
-		(diameter 0)
-		(color 0 0 0 0)
-	)
-	(junction
 		(at 139.7 66.04)
 		(diameter 0)
@@
 	)
 	(junction
+		(at 64.77 205.74)
+		(diameter 0)
+		(color 0 0 0 0)
+	)
+	(junction
 		(at 342.9 60.96)
 		(diameter 0)
@@
 	)
 	(junction
-		(at 64.77 180.34)
-		(diameter 0)
-		(color 0 0 0 0)
-	)
-	(junction
 		(at 374.65 86.36)
 		(diameter 0)
@@
 	)
 	(junction
+		(at 64.77 182.88)
+		(diameter 0)
+		(color 0 0 0 0)
+	)
+	(junction
 		(at 412.75 40.64)
 		(diameter 0)
@@
 	(wire
 		(pts
-			(xy 107.95 187.96) (xy 107.95 193.04)
+			(xy 107.95 190.5) (xy 107.95 193.04)
 		)
 		(stroke
@@
 	(wire
 		(pts
+			(xy 107.95 198.12) (xy 107.95 196.85)
+		)
+		(stroke
+			(width 0)
+			(type default)
+		)
+	)
+	(wire
+		(pts
 			(xy 488.95 86.36) (xy 508 86.36)
 		)
@@
 	(wire
 		(pts
+			(xy 107.95 196.85) (xy 119.38 196.85)
+		)
+		(stroke
+			(width 0)
+			(type default)
+		)
+	)
+	(wire
+		(pts
 			(xy 450.85 50.8) (xy 469.9 50.8)
 		)
@@
 	(wire
 		(pts
-			(xy 100.33 196.85) (xy 119.38 196.85)
+			(xy 100.33 196.85) (xy 107.95 196.85)
 		)
 		(stroke
@@
 	(wire
 		(pts
-			(xy 119.38 204.47) (xy 64.77 204.47)
+			(xy 107.95 205.74) (xy 64.77 205.74)
 		)
 		(stroke
@@
 	(wire
 		(pts
-			(xy 64.77 204.47) (xy 64.77 246.38)
+			(xy 64.77 134.62) (xy 64.77 182.88)
 		)
 		(stroke
@@
 	(wire
 		(pts
-			(xy 64.77 134.62) (xy 64.77 180.34)
-		)
-		(stroke
-			(width 0)
-			(type default)
-		)
-	)
-	(wire
-		(pts
 			(xy 171.45 43.18) (xy 171.45 40.64)
 		)
@@
 	(wire
 		(pts
-			(xy 107.95 180.34) (xy 64.77 180.34)
+			(xy 107.95 182.88) (xy 64.77 182.88)
 		)
 		(stroke
@@
 	(wire
 		(pts
-			(xy 64.77 180.34) (xy 64.77 204.47)
-		)
-		(stroke
-			(width 0)
-			(type default)
-		)
-	)
-	(wire
-		(pts
 			(xy 469.9 40.64) (xy 488.95 40.64)
 		)
@@
 	(wire
 		(pts
+			(xy 64.77 205.74) (xy 64.77 246.38)
+		)
+		(stroke
+			(width 0)
+			(type default)
+		)
+	)
+	(wire
+		(pts
 			(xy 527.05 106.68) (xy 527.05 109.22)
 		)
@@
 	(wire
 		(pts
+			(xy 64.77 182.88) (xy 64.77 205.74)
+		)
+		(stroke
+			(width 0)
+			(type default)
+		)
+	)
+	(wire
+		(pts
 			(xy 374.65 132.08) (xy 393.7 132.08)
 		)
@@
 	(symbol
 		(lib_id "Device:C")
-		(at 119.38 200.66 0)
+		(at 107.95 201.93 0)
 		(unit 1)
 		(exclude_from_sim no)
@@
 		(fields_autoplaced yes)
 		(property "Reference" "C2"
-			(at 123.19 199.3899 0)
+			(at 111.76 200.6599 0)
 			(effects
 				(font
@@
 		)
 		(property "Value" "C"
-			(at 123.19 201.9299 0)
+			(at 111.76 203.1999 0)
 			(effects
 				(font
@@
 		)
 		(property "Footprint" "Capacitor_SMD:C_0201_0603Metric"
-			(at 120.3452 204.47 0)
+			(at 108.9152 205.74 0)
 			(effects
 				(font
@@
 		)
 		(property "Datasheet" "~"
-			(at 119.38 200.66 0)
+			(at 107.95 201.93 0)
 			(effects
 				(font
@@
 		)
 		(property "Description" "Unpolarized capacitor"
-			(at 119.38 200.66 0)
+			(at 107.95 201.93 0)
 			(effects
 				(font
@@
 	(symbol
 		(lib_id "Device:C")
-		(at 107.95 184.15 0)
+		(at 107.95 186.69 0)
 		(unit 1)
 		(exclude_from_sim no)
@@
 		(fields_autoplaced yes)
 		(property "Reference" "C1"
-			(at 111.76 182.8799 0)
+			(at 111.76 185.4199 0)
 			(effects
 				(font
@@
 		)
 		(property "Value" "C"
-			(at 111.76 185.4199 0)
+			(at 111.76 187.9599 0)
 			(effects
 				(font
@@
 		)
 		(property "Footprint" "Capacitor_SMD:C_0201_0603Metric"
-			(at 108.9152 187.96 0)
+			(at 108.9152 190.5 0)
 			(effects
 				(font
@@
 		)
 		(property "Datasheet" "~"
-			(at 107.95 184.15 0)
+			(at 107.95 186.69 0)
 			(effects
 				(font
@@
 		)
 		(property "Description" "Unpolarized capacitor"
-			(at 107.95 184.15 0)
+			(at 107.95 186.69 0)
 			(effects
 				(font
