File: single-color/boards/Y43/Y42_routed_v4.kicad_pcb (KiCad board)
At the start: 4 copper layers, 42 x 51.2 mm, 197 parts, among them J1 LiPo, J1B LiPo, J2 UPDI pogo pads 1.27 mm (RESET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, M0 LED white 0402, M1 LED white 0402, M10 LED white 0402, M11 LED white 0402, M12 LED white 0402, M13 LED white 0402, M14 LED white 0402, M15 LED white 0402, M16 LED white 0402, M17 LED white 0402, M18 LED white 0402, M19 LED white 0402, M2 LED white 0402, M20 LED white 0402, M21 LED white 0402, M22 LED white 0402, M23 LED white 0402, M24 LED white 0402, M25 LED white 0402, M26 LED white 0402, M27 LED white 0402, M28 LED white 0402, M29 LED white 0402, M3 LED white 0402, M30 LED white 0402, M31 LED white 0402, M32 LED white 0402, M33 LED white 0402, M34 LED white 0402, M35 LED white 0402, M36 LED white 0402, M37 LED white 0402, M38 LED white 0402, M39 LED white 0402, M4 LED white 0402, M40 LED white 0402, M41 LED white 0402, M42 LED white 0402, M43 LED white 0402, M44 LED white 0402, M45 LED white 0402, M46 LED white 0402, M47 LED white 0402, M48 LED white 0402, M49 LED white 0402, M5 LED white 0402, M50 LED white 0402, M51 LED white 0402, M52 LED white 0402, M53 LED white 0402, M54 LED white 0402, M55 LED white 0402, M56 LED white 0402, M57 LED white 0402, M58 LED white 0402, M59 LED white 0402, M6 LED white 0402, M7 LED white 0402, M8 LED white 0402, M9 LED white 0402, SW1 SW_Push, SW2 SW_Push, U1 AVR128DB48-I/6LX, U2 LIS2DW12TR, U4 BQ25570RGRR, Y1 32.768kHz

Commit message: single-color: schematic regenerated to match Y42 v4; re-apply lost pad-landing and silk fixes; fab files re-exported
- gen_schematic.py: 7 mode LEDs (IND7 = ALM), BZ1 piezo on BUZ_A/BUZ_B (PB4/PB5), RESET (PF6) to pogo pad 1, 4-pad pogo J2, dummy resistors R61-R67, SC1+/SC1- cell pads; watch_solar.kicad_sch regenerated. Netlist == board (197 parts, 0 differences apart from the far KMR2 switch pads).
- Y42_routed_v4: IND7 value ALM; pad/via landing stubs, silk dashes removed, silk 0.15 mm, two-line mode labels re-applied (v4 had lost them), ground zone refilled. DRC 0 errors / 0 unconnected.
- fab42/ and Y42_routed_v4_gerbers.zip re-exported, BOM/CPL regenerated, renders, DECISION-LOG and PRE-ORDER-CHECKLIST updated.

Co-Authored-By: Claude Sonnet 5.5 <noreply@anthropic.com>
Parts:
- IND7: value LCK -> ALM
Routing:
- net GND: track 10.0 -> 32.8 mm
- net +3V3: track 42.3 -> 48.7 mm
- net VBAT: track 48.2 -> 54.6 mm
- net /ROW11: track 33.5 -> 38.1 mm
- net /SOLAR_IN: track 9.61 -> 13.0 mm
- net /BUZ_A: track 30.4 -> 32.5 mm
- net /BUZ_B: track 29.3 -> 31.3 mm
- net /ROW2: track 119.7 -> 121.7 mm
- net /VOUT_SET: track 4.64 -> 6.62 mm
- net /OK_PROG: track 9.83 -> 11.8 mm
- net /BATT: track 49.0 -> 50.8 mm
- net /VRDIV: track 5.83 -> 7.61 mm
- net /LBUCK: track 15.7 -> 17.4 mm
- net /LBOOST: track 4.81 -> 6.49 mm
- net /VBAT_OV: track 1.53 -> 3.00 mm
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Other:
- board text added: "ALM"
- board text added: "BAT"
- board text added: "CFG"
- board text added: "F"
- board text added: "FUN"
- board text added: "LCK"
- board text added: "M"
- board text added: "S"
- board text added: "SET"
- board text added: "T"
- board text added: "TMR"
- board text added: "W"
- board text removed: "ALM-T"
- board text removed: "BAT-W"
- board text removed: "CFG-F"
- board text removed: "FUN-T"
- board text removed: "LCK-S"
- board text removed: "SET-S"
- board text removed: "TMR-M"
