File: single-color/schematic/watch_solar.kicad_sch (KiCad schematic)
At the start: 190 parts, among them J1 LiPo, J1B LiPo 2, J2 UPDI Tag-Connect TC2030-NL, J3 Solar cell KXOB25-05X3TF, M0 LED white 0402, M1 LED white 0402, M10 LED white 0402, M11 LED white 0402, M12 LED white 0402, M13 LED white 0402, M14 LED white 0402, M15 LED white 0402, M16 LED white 0402, M17 LED white 0402, M18 LED white 0402, M19 LED white 0402, M2 LED white 0402, M20 LED white 0402, M21 LED white 0402, M22 LED white 0402, M23 LED white 0402, M24 LED white 0402, M25 LED white 0402, M26 LED white 0402, M27 LED white 0402, M28 LED white 0402, M29 LED white 0402, M3 LED white 0402, M30 LED white 0402, M31 LED white 0402, M32 LED white 0402, M33 LED white 0402, M34 LED white 0402, M35 LED white 0402, M36 LED white 0402, M37 LED white 0402, M38 LED white 0402, M39 LED white 0402, M4 LED white 0402, M40 LED white 0402, M41 LED white 0402, M42 LED white 0402, M43 LED white 0402, M44 LED white 0402, M45 LED white 0402, M46 LED white 0402, M47 LED white 0402, M48 LED white 0402, M49 LED white 0402, M5 LED white 0402, M50 LED white 0402, M51 LED white 0402, M52 LED white 0402, M53 LED white 0402, M54 LED white 0402, M55 LED white 0402, M56 LED white 0402, M57 LED white 0402, M58 LED white 0402, M59 LED white 0402, M6 LED white 0402, M7 LED white 0402, M8 LED white 0402, M9 LED white 0402, SW1 SW_Push, SW2 SW_Push, U1 AVR128DB48-I/6LX, U2 LIS2DW12TR, U4 BQ25570RGRR, Y1 32.768kHz

Commit message: single-color: schematic regenerated to match Y42 v4; re-apply lost pad-landing and silk fixes; fab files re-exported
- gen_schematic.py: 7 mode LEDs (IND7 = ALM), BZ1 piezo on BUZ_A/BUZ_B (PB4/PB5), RESET (PF6) to pogo pad 1, 4-pad pogo J2, dummy resistors R61-R67, SC1+/SC1- cell pads; watch_solar.kicad_sch regenerated. Netlist == board (197 parts, 0 differences apart from the far KMR2 switch pads).
- Y42_routed_v4: IND7 value ALM; pad/via landing stubs, silk dashes removed, silk 0.15 mm, two-line mode labels re-applied (v4 had lost them), ground zone refilled. DRC 0 errors / 0 unconnected.
- fab42/ and Y42_routed_v4_gerbers.zip re-exported, BOM/CPL regenerated, renders, DECISION-LOG and PRE-ORDER-CHECKLIST updated.

Co-Authored-By: Claude Sonnet 5.5 <noreply@anthropic.com>
Parts:
- removed C60, C61, C62: 100n, Capacitor_SMD:C_0402_1005Metric, symbol Device:C
- removed J2: UPDI Tag-Connect TC2030-NL, Connector:Tag-Connect_TC2030-IDC-NL_2x03_P1.27mm_Vertical, symbol Connector_Generic:Conn_02x03_Odd_Even
- removed J3: Solar cell KXOB25-05X3TF, Connector_PinHeader_2.54mm:PinHeader_1x02_P2.54mm_Vertical, symbol Connector_Generic:Conn_01x02
- added BZ1: PKMCS0909E4000-R1, LEDWatch:Piezo_Murata_PKMCS0909E4000-R1_9x9mm, symbol Device:Buzzer
- added IND7: ALM, LED_SMD:LED_0402_1005Metric, symbol Device:LED
- added J2: UPDI pogo pads 1.27 mm (RESET VDD GND UPDI), LEDWatch:UPDI_Pogo_1x4_P1.27mm_2Guide, symbol Connector_Generic:Conn_01x04
- added R61, R62, R63, R64, R65, R66, R67: 10k, Resistor_SMD:R_0402_1005Metric, symbol Device:R
- added SC1+, SC1-: cell pad, LEDWatch:KXOB25_cell_pad_2.5x7.4mm, symbol Connector:TestPoint
- IND1: value LED white 0402 (indicator) -> SET
- IND2: value LED white 0402 (indicator) -> TMR
- IND3: value LED white 0402 (indicator) -> BAT
- IND4: value LED white 0402 (indicator) -> FUN
- IND5: value LED white 0402 (indicator) -> CFG
- IND6: value LED white 0402 (indicator) -> LCK
- J1B: value LiPo 2 -> LiPo
Connections:
- net COL6: now also IND7.2 (A)
- net GND: now also J2.3 (Pin_3), SC1-.1
- net ROW11: now also IND7.1 (K)
- net SOLAR_IN: now also SC1+.1
- net UPDI: now also J2.4 (Pin_4)
- net VBAT: now also J2.2 (Pin_2)
- net RESET: now reaches U1.40 (~{RESET}/PF6)
- net RESET: now also J2.1 (Pin_1)
- net BUZ_A: now reaches U1.8 (PB4)
- net BUZ_A: now also BZ1.1 (+)
- net BUZ_B: now reaches U1.9 (PB5)
- net BUZ_B: now also BZ1.2 (-)
- no-connect marks 25 -> 27
Other:
- note added: "Piezo BZ1: PB4 / PB5 drive it in antiphase (TCA1 split mode, PB5 inverted via PORTB.PIN5CTRL.INVEN)"
- note added: "UPDI programming pads (1.27 mm pogo row, back side): 1 RESET, 2 VBAT, 3 GND, 4 UPDI"
- note removed: "UPDI programming (Tag-Connect TC2030-IDC-NL): pad1 UPDI, pad2 VBAT, pad6 GND"
