File: rgb/LED Watch - RGB.kicad_sch (KiCad schematic)
At the start: 146 parts, among them J1 AVR-ISP-6, J2 Lipo, J3 Coin Cell, SW1 SW_DPST, SW2 SW_DPST, U10 B39D3RGB-F6C0001HOU1930, U100 B39D3RGB-F6C0001HOU1930, U101 B39D3RGB-F6C0001HOU1930, U102 B39D3RGB-F6C0001HOU1930, U103 B39D3RGB-F6C0001HOU1930, U104 B39D3RGB-F6C0001HOU1930, U105 B39D3RGB-F6C0001HOU1930, U106 B39D3RGB-F6C0001HOU1930, U107 B39D3RGB-F6C0001HOU1930, U108 B39D3RGB-F6C0001HOU1930, U109 B39D3RGB-F6C0001HOU1930, U11 B39D3RGB-F6C0001HOU1930, U110 B39D3RGB-F6C0001HOU1930, U111 B39D3RGB-F6C0001HOU1930, U112 B39D3RGB-F6C0001HOU1930, U113 B39D3RGB-F6C0001HOU1930, U114 B39D3RGB-F6C0001HOU1930, U115 B39D3RGB-F6C0001HOU1930, U116 B39D3RGB-F6C0001HOU1930, U117 B39D3RGB-F6C0001HOU1930, U118 B39D3RGB-F6C0001HOU1930, U119 B39D3RGB-F6C0001HOU1930, U12 B39D3RGB-F6C0001HOU1930, U120 B39D3RGB-F6C0001HOU1930, U121 B39D3RGB-F6C0001HOU1930, U122 B39D3RGB-F6C0001HOU1930, U123 B39D3RGB-F6C0001HOU1930, U124 B39D3RGB-F6C0001HOU1930, U125 B39D3RGB-F6C0001HOU1930, U126 B39D3RGB-F6C0001HOU1930, U127 B39D3RGB-F6C0001HOU1930, U128 B39D3RGB-F6C0001HOU1930, U129 B39D3RGB-F6C0001HOU1930, U13 B39D3RGB-F6C0001HOU1930, U130 B39D3RGB-F6C0001HOU1930, U131 B39D3RGB-F6C0001HOU1930, U132 B39D3RGB-F6C0001HOU1930, U133 B39D3RGB-F6C0001HOU1930, U134 BMI160, U135 ATmega165PA-M, U14 B39D3RGB-F6C0001HOU1930, U15 B39D3RGB-F6C0001HOU1930, U16 B39D3RGB-F6C0001HOU1930, U17 B39D3RGB-F6C0001HOU1930, U18 B39D3RGB-F6C0001HOU1930, U19 B39D3RGB-F6C0001HOU1930, U2 B39D3RGB-F6C0001HOU1930, U20 B39D3RGB-F6C0001HOU1930, U21 B39D3RGB-F6C0001HOU1930, U22 B39D3RGB-F6C0001HOU1930, U23 B39D3RGB-F6C0001HOU1930, U24 B39D3RGB-F6C0001HOU1930, U25 B39D3RGB-F6C0001HOU1930, U26 B39D3RGB-F6C0001HOU1930, U27 B39D3RGB-F6C0001HOU1930, U28 B39D3RGB-F6C0001HOU1930, U29 B39D3RGB-F6C0001HOU1930, U3 B39D3RGB-F6C0001HOU1930, U30 B39D3RGB-F6C0001HOU1930, U31 B39D3RGB-F6C0001HOU1930, U32 B39D3RGB-F6C0001HOU1930, U33 B39D3RGB-F6C0001HOU1930, U34 B39D3RGB-F6C0001HOU1930, U35 B39D3RGB-F6C0001HOU1930, U36 B39D3RGB-F6C0001HOU1930, U37 B39D3RGB-F6C0001HOU1930, U38 B39D3RGB-F6C0001HOU1930, U39 B39D3RGB-F6C0001HOU1930, U4 B39D3RGB-F6C0001HOU1930, U40 B39D3RGB-F6C0001HOU1930, U41 B39D3RGB-F6C0001HOU1930, U42 B39D3RGB-F6C0001HOU1930, U43 B39D3RGB-F6C0001HOU1930, U44 B39D3RGB-F6C0001HOU1930, U45 B39D3RGB-F6C0001HOU1930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

Commit message: rgb: the live RGB work (Oct 2026 edits) becomes the main "LED Watch - RGB" project; add fab-rfq 2026-10-05, snapshots, Rhino layout
- rgb/LED Watch - RGB.* = the files from the working folder as of 2026-10-14 (board routes with 0 unconnected nets); the December 2025 version that the repository had is kept in rgb/archive/pre-claude/2025-12-08 ...
- rgb/production/fab-rfq 2026-10-05/ (BOM, placement files, Gerbers, DRC, quote screenshots, notes), rgb/archive/pre-claude/2026-10-05 snapshots ..., rgb/mechanical/watch layout 1.3dm
- updated KiCad project/layout state files of the archived variants from the working folder
- .gitignore: _old-desktop-copies/ (the previous loose Desktop copies, kept untouched next to the repository)

Co-Authored-By: Claude Sonnet 5.5 <noreply@anthropic.com>
Parts:
- U134: value BMI160 -> BMI270
Changed lines of the file:
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@@
 			)
 		)
-		(property "Value" "BMI160"
+		(property "Value" "BMI270"
 			(at 52.9433 278.13 0)
 			(effects
@@
 			)
 		)
-		(property "Datasheet" "https://www.bosch-sensortec.com/media/boschsensortec/downloads/datasheets/bst-bmi160-ds000.pdf"
+		(property "Datasheet" "https://www.bosch-sensortec.com/media/boschsensortec/downloads/datasheets/bst-bmi270-ds000.pdf"
 			(at 33.02 266.7 0)
 			(effects
@@
 			)
 		)
-		(property "Description" "Small, low power inertial measurement unit, LGA-14"
+		(property "Description" "Bosch BMI270 6-axis IMU (accel+gyro), LGA-14 2.5x3.0mm; pin-compatible successor to BMI160 (symbol drawn from BMI160, identical pin-out)"
 			(at 50.8 288.29 0)
 			(effects
